Commit message: Add files via upload

File: robo_nemotron_description/urdf/robo_nemotron_1.urdf (robot description, URDF)
Before this commit: robot robo_nemotron, 8 links, 7 joints
Links:
- removed link world
- link base_link: mass 2.0 -> None
- link gripper_base: mass 0.3 -> None
- link left_finger: mass 0.1 -> None
- link link_1: mass 1.0 -> None
- link link_2: mass 0.8 -> None
- link link_3: mass 0.5 -> None
- link right_finger: mass 0.1 -> None
Joints:
- removed joint world_fixed_joint
